File: CAD/PCB/Reverb.kicad_pcb (KiCad board)
At the start: 2 copper layers, 82.6 x 74.3 mm, 109 parts, among them J1 USB_C_Receptacle_PowerOnly_6P, J10 Conn_01x08, J11 Conn_01x03, J12 Conn_01x06, J2 USB_C_Receptacle_PowerOnly_6P, J3 Conn_01x03, J4 Conn_01x05, J5 Conn_01x03, J6 Conn_01x02, J7 USB_C_Receptacle_USB2.0_16P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

Commit message: Added code
Parts:
- added C33: 1uF, Capacitor_SMD:C_0603_1608Metric, F.Cu at (142.0, 70.9)
- added D28: 1N4148W, Diode_SMD:D_SOD-123, F.Cu at (145.2, 70.2)
- added R11: 10k, Resistor_SMD:R_0603_1608Metric, F.Cu at (144.3, 72.2)
- added R12: 10k, Resistor_SMD:R_0603_1608Metric, F.Cu at (144.3, 68.2)
Connections:
- J8 pad 1: Net-(J8-Pin_1) -> GND
- J8 pad 2: GND -> Net-(J8-Pin_2)
- SW1 pad 2: Net-(J8-Pin_1) -> Net-(J8-Pin_2)
- U1 pad 25: unconnected-(U1-IO48-Pad25) -> /Pixel Data
- U1 pad 4: /Pixel Data -> /VolumeTap
Routing:
- net Net-(D28-A): track 20.0 -> 49.1 mm, vias 0 -> 2
- net /VolumeTap: track 0.00 -> 27.8 mm, vias 0 -> 2
- net Net-(J8-Pin_2): track 0.00 -> 7.71 mm
- net Net-(J8-Pin_1): track 5.71 -> 0.00 mm
- net GND: track 49.8 -> 54.9 mm, vias 15 -> 13
- net Net-(D28-K): track 0.00 -> 2.70 mm
- net +3.3V: track 145.9 -> 147.0 mm
- net /VSENSE: track 28.7 -> 29.6 mm
- net /Pixel Data: vias 5 -> 4
- net Net-(J6-Pin_2): vias 0 -> 2
