File: CAD/PCB/Reverb.kicad_sch (KiCad schematic)
At the start: 99 parts, among them J1 USB_C_Receptacle_PowerOnly_6P, J10 Conn_01x08, J11 Conn_01x03, J12 Conn_01x06, J2 USB_C_Receptacle_PowerOnly_6P, J3 Conn_01x03, J4 Conn_01x05, J5 Conn_01x03, J6 Conn_01x02, J7 USB_C_Receptacle_USB2.0_16P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

Commit message: Added code
Parts:
- added C33: 1uF, Capacitor_SMD:C_0603_1608Metric, symbol Device:C_Small
- added D28: 1N4148W, Diode_SMD:D_SOD-123, symbol Diode:1N4148W
- added R11, R12: 10k, Resistor_SMD:R_0603_1608Metric, symbol Device:R
Connections:
- net GND: now also J8.1 (Pin_1), C33.1, R12.1; no longer J8.2 (Pin_2)
- net Pixel Data: now also U1.25 (IO48); no longer U1.4 (IO4)
- net at J6.1 (Pin_1), U2.9 (OUTP): now also D28.2 (A)
- net at SW1.2 (B): now also J8.2 (Pin_2); no longer J8.1 (Pin_1)
- new net: D28.1 (K), R11.2
- new net VolumeTap: C33.2, R11.1, R12.2, U1.4 (IO4)
Other:
- moved on the sheet: C1, C10, C11, C12, C13, C14, C15, C16, C17, C18, C19, C2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
